File: hw-chipdown/PicoGUS chipdown.kicad_sch (KiCad schematic)
At the start: 65 parts, among them J1 Bus_ISA_8bit, J10 Conn_01x02_Pin, J2 DEBUG, J3 IRQDMA_JP, J4 UART_TX, J5 USB_A - joy, J7 3.5mm TRS, J8 Wavetable, J9 3.5mm TRS, Q1 AO3401A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

Commit message: v2.0 with 0805 components
Parts:
- C10: footprint Capacitor_SMD:C_0603_1608Metric -> Capacitor_SMD:C_0805_2012Metric_Pad1.18x1.45mm_HandSolder
- C2, C23, C3, C4, C45, C5, C6, C7, C8, C9: footprint Capacitor_SMD:C_0402_1005Metric -> Capacitor_SMD:C_0805_2012Metric_Pad1.18x1.45mm_HandSolder
- C? (x2): footprint Capacitor_SMD:C_0805_2012Metric -> Capacitor_SMD:C_0805_2012Metric_Pad1.18x1.45mm_HandSolder
- D1: footprint LED_SMD:LED_0603_1608Metric -> LED_SMD:LED_0805_2012Metric_Pad1.15x1.40mm_HandSolder
- F1: footprint Fuse:Fuse_1206_3216Metric -> Fuse:Fuse_1206_3216Metric_Pad1.42x1.75mm_HandSolder
- FB1, FB2, FB3, FB4: footprint Inductor_SMD:L_0805_2012Metric -> Inductor_SMD:L_0805_2012Metric_Pad1.15x1.40mm_HandSolder
- R1, R13, R17, R18, R4, R5, R6, R7, R8, R9: footprint Resistor_SMD:R_0402_1005Metric -> Resistor_SMD:R_0805_2012Metric_Pad1.20x1.40mm_HandSolder
- R2, R3: footprint Resistor_SMD:R_0805_2012Metric -> Resistor_SMD:R_0805_2012Metric_Pad1.20x1.40mm_HandSolder
- SW1: footprint Button_Switch_SMD:SW_SPST_TL3305A -> footprints:SW_SPST_PTS810_handsoldering
